File: 6vleadacidsolar.sch (KiCad schematic (older format))
At the start: 61 parts, among them J1 CONN2, J2 CONN2, J3 CONN4, J4 CONN6, J5 CONN3, J6 CONN3, J7 CONN3, Q1 SI2369, Q2 MMBT4401, Q3 MMBT4403, Q4 MMBT4401, Q5 SI2369, Q6 MMBT4401, Q7 SI2369, Q8 MMBT4401, U1 CS30CL, U2 CS30CL

Commit message: Schematic cleanup, add part numbers to parts in schematic
Parts:
- C1, C2: MFG UNITED CHEMI-CON -> (none); MPN EMZJ160ADR471MHA0G -> (none); PartNumber (none) -> 800009-477
- C10, C11, C12, C13, C14, C15, C17, C18, C3, C5, C6, C9: PartNumber (none) -> 800000-104
- C7: PartNumber (none) -> 800002-471
- C8: PartNumber (none) -> 800003-106
- CR2, CR3: MFG VISHAY -> (none); MPN ES1A-E3/61T -> (none); PartNumber (none) -> 800109-101
- CR4: symbol ZENER -> ZENER-RESCUE-6vleadacidsolar; MFG ON SEMI -> (none); MPN 1SMA13AT3G -> (none); PartNumber (none) -> 800132-013
- CR5: PartNumber (none) -> 800127-101
- F1: MFG TE -> (none); MPN MINISMD160F -> (none); PartNumber (none) -> 800133-110
- J1, J2: PartNumber (none) -> 800114-102
- J3: PartNumber (none) -> 800114-104
- J4: PartNumber (none) -> 800114-106
- J5, J6, J7: PartNumber (none) -> 800114-103
- L1: MFG BOURNS -> (none); MPN SDE0805A-470K -> (none); PartNumber (none) -> 800101-047
- Q1, Q5, Q7: MFG VISHAY -> (none); MPN SI2369DS-T1-E3 -> (none); PartNumber (none) -> 800134-101
- Q2, Q4, Q6, Q8: PartNumber (none) -> 800110-101
- Q3: PartNumber (none) -> 800111-101
- R1, R9: MFG SUSUMU -> (none); MPN KRL1220E-M-R039-F-T5 -> (none); PartNumber (none) -> 800018-039
- R10, R11, R12, R14, R16: PartNumber (none) -> 800010-104
- R13, R15, R8: PartNumber (none) -> 800010-472
- R2: PartNumber (none) -> 800010-100
- R3, R6, R7: PartNumber (none) -> 800023-100
- R4: PartNumber (none) -> 800023-200
- R5: PartNumber (none) -> 800010-102
- U1, U2: MFG ST -> (none); MPN CS30CL -> (none); PartNumber (none) -> 800122-101
- VR1: PartNumber (none) -> 800105-101
Other:
- moved on the sheet: C12, C13, C14, C15, J5, J6, J7, Q5, Q6, R10, R13, SJ1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
